File: M304N.kicad_sch (KiCad schematic)
At the start: 3 parts, among them IC1 TEENSY_4.1, J1 USB_A

Commit message: RESET/PRGスイッチ追加
Parts:
- added SW1: RESET, symbol Switch:SW_Push
- added SW2: PRG, symbol Switch:SW_Push
Connections:
- net GND: now also SW1.2, SW2.2
- net at IC1.46 (PROGRAM): now also SW2.1
- net at IC1.47 (ON/OFF): now also SW1.1

Commit message: RELAYユニットに逆転制御を含んだサンプル回路を記した．
Other:
- added sheet WINDOW MOTOR UNIT (window_motor_unit.kicad_sch)
- sheet RELAY UNIT ports: added 12V, 24V, 3.3V, 5V, GND; removed none
Changed lines of the file:
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@@
+	)
+	(sheet
+		(at 179.07 142.24)
+		(size 19.685 12.7)
+		(exclude_from_sim no)
+		(in_bom yes)
+		(on_board yes)
+		(dnp no)
+		(fields_autoplaced yes)
+		(stroke
+			(width 0.1524)
+			(type solid)
+		)
+		(fill
+			(color 0 0 0 0)
+		)
+		(property "Sheetname" "WINDOW MOTOR UNIT"
+			(at 179.07 141.5284 0)
+			(show_name no)
+			(do_not_autoplace no)
+			(effects
+				(font
+					(size 1.27 1.27)
+				)
+				(justify left bottom)
+			)
+		)
+		(property "Sheetfile" "window_motor_unit.kicad_sch"
+			(at 179.07 155.5246 0)
+			(show_name no)
+			(do_not_autoplace no)
+			(effects
+				(font
+					(size 1.27 1.27)
+				)
+				(justify left top)
+			)
+		)
+		(instances
+			(project "M304N"
+				(path "/c41feddf-9b57-4156-a07a-047a9379ecf1"
+					(page "4")
+				)
+			)
+		)
 	)
 	(sheet
@@
 	(sheet
 		(at 219.456 126.238)
-		(size 42.418 22.606)
+		(size 28.194 22.606)
 		(exclude_from_sim no)
 		(in_bom yes)
@@
 			)
 		)
+		(pin "3.3V" input
+			(at 219.456 132.08 180)
+			(effects
+				(font
+					(size 1.27 1.27)
+				)
+				(justify left)
+			)
+		)
+		(pin "5V" input
+			(at 219.456 134.62 180)
+			(effects
+				(font
+					(size 1.27 1.27)
+				)
+				(justify left)
+			)
+		)
+		(pin "12V" input
+			(at 219.456 137.16 180)
+			(effects
+				(font
+					(size 1.27 1.27)
+				)
+				(justify left)
+			)
+		)
+		(pin "24V" input
+			(at 219.456 139.7 180)
+			(effects
+				(font
+					(size 1.27 1.27)
+				)
+				(justify left)
+			)
+		)
+		(pin "GND" input
+			(at 219.456 145.415 180)
+			(effects
+				(font
+					(size 1.27 1.27)
+				)
+				(justify left)
+			)
+		)
